File: stm32f1 blue pill/Rev STM32f1 Kicad/Rev STM32f1 Kicad.kicad_sch (KiCad schematic)
At the start: 10 parts, among them U1 STM32F103C8T6

Commit message: updated
Parts:
- added C9: 100n, symbol Device:C_Small
- added R1: 10k, symbol Device:R_Small
- added SW1: SW_SPDT, symbol Switch:SW_SPDT
Connections:
- net +3.3V: now also SW1.3 (C)
- net GND: now also C9.2, SW1.1 (A)
- net BOOT0: now reaches U1.44 (BOOT0)
- net BOOT0: now also R1.2
- net NRST: now reaches U1.7 (NRST)
- net NRST: now also C9.1
- new net: R1.1, SW1.2 (B)
