File: stm32wb55-RF/Bluetooth-wb55ceu/Bluetooth-wb55ceu.kicad_sch (KiCad schematic)
At the start: 45 parts, among them J1 USB_C_Receptacle_USB2.0_16P, J2 Conn_Coaxial, J3 Conn_01x04_Pin, J4 Conn_02x05_Odd_Even, SW1 SW_Push, SW2 SW_Push, U1 LM1117MP-3.3, U2 USBLC6-2SC6, U3 STM32WB55CEUx, Y1 32KHz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

Commit message: added tracec and vias
Parts:
- removed SW2: SW_Push, Button_Switch_SMD:SW_SPST_CK_RS282G05A3, symbol Switch:SW_Push
- removed Y2: 12MHz, Crystal:Crystal_HC49-4H_Vertical, symbol Device:Crystal
- added H1, H2, H3, H4: MountingHole_Pad, MountingHole:MountingHole_3.2mm_M3_Pad, symbol Mechanical:MountingHole_Pad
- added Y2: 12MHz, Crystal:Crystal_SMD_5032-4Pin_5.0x3.2mm, symbol Device:Crystal_GND24
- R1, R2, R3, R4, R5, R6, R7: footprint Resistor_SMD:R_0402_1005Metric -> Resistor_SMD:R_0805_2012Metric_Pad1.20x1.40mm_HandSolder
Connections:
- net GND: now also H1.1, H2.1, H3.1, H4.1, Y2.2, Y2.4
- net OSC_IN: now also Y2.1
- net OSC_OUT: now also Y2.3
- net D+: now reaches J1.A6 (D+), J1.B6 (D+), U2.1 (I/O1)
- net D-: now reaches J1.A7 (D-), J1.B7 (D-), U2.3 (I/O2)
- net at Y1.2: no longer Y1.3
- no-connect marks 23 -> 25
Other:
- note added: "Mounting Holes (M3)"
